File: kbd.kicad_sch (KiCad schematic)
At the start: 154 parts, among them J2 USB_C_Receptacle_USB2.0, SW1 ESC, SW10 A, SW11 BACKSLASH, SW12 SUPER, SW13 P, SW14 RSHIFT, SW15 TWO, SW16 W, SW17 S, SW18 Z, SW19 LALT, SW2 TAB, SW20 SEMICOLON, SW21 UP, SW22 THREE, SW23 E, SW24 D, SW25 X, SW26 SPACE, SW27 DOT, SW28 ENTER, SW29 FOUR, SW3 CAPS, SW30 R, SW31 F, SW32 C, SW33 ALTGR, SW34 SLASH, SW35 BACKSPACE, SW36 FIVE, SW37 T, SW38 G, SW39 V, SW4 LSHIFT, SW40 RALT, SW41 APOSTROPHE, SW42 F1, SW43 SIX, SW44 Y, SW45 H, SW46 B, SW47 FN, SW48 LSQUARE, SW49 F2, SW5 LCTRL, SW50 SEVEN, SW51 U, SW52 J, SW53 N, SW54 LEFT, SW55 DASH, SW56 F3, SW57 EIGHT, SW58 I, SW59 K, SW6 ZERO, SW60 M, SW61 DOWN, SW62 EQUAL, SW63 F4, SW64 NINE, SW65 O, SW66 L, SW67 COMMA, SW68 RIGHT, SW69 RSQUARE, SW7 HASH, SW70 RST, SW8 ONE, SW9 Q, U2 ATmega32U2-A, Y1 16MHz

Commit message: update
Parts:
- added J1: (no value), symbol Connector:Conn_01x06_Male
- D71: footprint LED_THT:LED_D3.0mm -> (none)
Connections:
- net COL1: now also J1.3 (Pin_3)
- net GND: now also J1.2 (Pin_2)
- net ROW5: now also J1.4 (Pin_4)
- net VCC: now also J1.1 (Pin_1)
- net RST: now reaches R2.2, SW70.2, U2.24 (PC1/~{RESET})
- net RST: now also J1.5 (Pin_5)
- net USB_P: now reaches J2.A6 (D+), J2.B6 (D+), R3.1
- net USB_N: now reaches J2.A7 (D-), J2.B7 (D-), R4.1
- net ROW6 renamed MOSI
- net MOSI: now also J1.6 (Pin_6)
Other:
- moved on the sheet: C1, C2, C3, C4, D70, D71, J2, R1, R2, R3, R4, R5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
